File: hw/ECE319K_Starter/ECE319K_Starter.kicad_sch (KiCad schematic)
At the start: 44 parts, among them J1 AudioJack, J2 Speaker, J3 UART1, J4 Pot, J6 GND, J7 DACOUT, SW1 UP, SW2 LEFT, SW3 DOWN, SW4 RGHT, U1 Adafruit ST7735R, U2 LP-MSPM0G3507, U3 MCP34119P, U4 HiLetGo_ST7735R

Commit message: lab 1 submission
lab 1 submission
Parts:
- added D4, D5: LED, ECE445L:LED_D5.0mm, symbol ECE445L:LED
- added R18, R19, R20, R21: 470, ECE445L:R_Axial_DIN0204_L3.6mm_D1.6mm_P7.62mm_Horizontal, symbol ECE445L:R_0.125W
- added SW5, SW6: RGHT, ECE445L:SW_PUSH_6mm, symbol ECE445L:SW_Push
Connections:
- net +3V3: now also SW5.2, SW6.1
- net GND: now also D4.1 (K), D5.1 (K), R19.1, R20.2
- net PB4: now also R18.2, R19.2, R21.1, SW5.1
- new net: D5.2 (A), R21.2
- new net: D4.2 (A), R18.1
- new net Pc7: R20.1, SW6.2
